File: PCB/KiCad/LumiTimeV2.kicad_pcb (KiCad board)
At the start: 2 copper layers, 35 x 35 mm, 54 parts, among them J1 Conn_06_Pin, U1 ATmega328-A, U2 PCF8563T, Y1 32,768 kHz

Commit message: Change#007
Some new ideas
Routing:
- net +3V7: track 70.9 -> 86.3 mm
Changed lines of the file:
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@@
 		)
 		(height 24)
-		(gr_text "35,00 mm"
+		(gr_text "35,0 mm"
 			(at 150 122.2 0)
 			(layer "Cmts.User")
@@
 			(units 3)
 			(units_format 1)
-			(precision 2)
+			(precision 1)
 		)
 		(style
@@
 	)
 	(segment
-		(start 143.585211 96.135211)
-		(end 143.585211 97.385211)
-		(width 0.4)
-		(layer "F.Cu")
-		(net 15)
-	)
-	(segment
 		(start 156.25 103.4)
 		(end 154.6 103.4)
-		(width 0.4)
+		(width 0.5)
 		(layer "F.Cu")
 		(net 15)
@@
 		(start 156 87.25)
 		(end 154.85 87.25)
-		(width 0.4)
-		(layer "F.Cu")
-		(net 15)
-	)
-	(segment
-		(start 143 93.947316)
-		(end 143 95.55)
+		(width 0.5)
+		(layer "F.Cu")
+		(net 15)
+	)
+	(segment
+		(start 150.75 91)
+		(end 151.75 92)
+		(width 0.4)
+		(layer "F.Cu")
+		(net 15)
+	)
+	(segment
+		(start 143.2 99.55)
+		(end 142.9 99.85)
 		(width 0.4)
 		(layer "F.Cu")
@@
 		(start 157.5 86.25)
 		(end 157 86.25)
-		(width 0.4)
-		(layer "F.Cu")
-		(net 15)
-	)
-	(segment
-		(start 143.76 97.56)
-		(end 145.025 97.56)
-		(width 0.4)
+		(width 0.5)
 		(layer "F.Cu")
 		(net 15)
@@
 		(start 153.1 104.9)
 		(end 153.1 107)
-		(width 0.4)
+		(width 0.5)
 		(layer "F.Cu")
 		(net 15)
@@
 		(start 154.85 87.25)
 		(end 153.2 88.9)
-		(width 0.4)
-		(layer "F.Cu")
-		(net 15)
-	)
-	(segment
-		(start 143.15 95.7)
-		(end 143.585211 96.135211)
+		(width 0.5)
+		(layer "F.Cu")
+		(net 15)
+	)
+	(segment
+		(start 145.947316 91)
+		(end 150.75 91)
+		(width 0.4)
+		(layer "F.Cu")
+		(net 15)
+	)
+	(segment
+		(start 143.2 97.7)
+		(end 143.2 99)
 		(width 0.4)
 		(layer "F.Cu")
@@
 		(start 153.2 90.55)
 		(end 151.75 92)
-		(width 0.4)
-		(layer "F.Cu")
-		(net 15)
-	)
-	(segment
-		(start 151.75 92)
-		(end 150.75 91)
+		(width 0.5)
+		(layer "F.Cu")
+		(net 15)
+	)
+	(segment
+		(start 142.9 101.8)
+		(end 142.9 102.5)
 		(width 0.4)
 		(layer "F.Cu")
@@
 		(start 157 86.25)
 		(end 156 87.25)
-		(width 0.4)
-		(layer "F.Cu")
-		(net 15)
-	)
-	(segment
-		(start 143 95.55)
+		(width 0.5)
+		(layer "F.Cu")
+		(net 15)
+	)
+	(segment
+		(start 145.3 104.9)
+		(end 153.1 104.9)
+		(width 0.4)
+		(layer "F.Cu")
+		(net 15)
+	)
+	(segment
+		(start 143.2 98.35)
+		(end 143.2 99.55)
+		(width 0.4)
+		(layer "F.Cu")
+		(net 15)
+	)
+	(segment
+		(start 143.2 95.75)
 		(end 143.15 95.7)
-		(width 0.3)
-		(layer "F.Cu")
-		(net 15)
-	)
-	(segment
-		(start 143.585211 98.085211)
-		(end 144.75 99.25)
-		(width 0.4)
-		(layer "F.Cu")
-		(net 15)
-	)
-	(segment
-		(start 150.75 91)
-		(end 145.947316 91)
-		(width 0.4)
-		(layer "F.Cu")
-		(net 15)
-	)
-	(segment
-		(start 143.585211 97.385211)
-		(end 143.76 97.56)
-		(width 0.4)
-		(layer "F.Cu")
-		(net 15)
-	)
-	(segment
-		(start 145.947316 91)
-		(end 143 93.947316)
+		(width 0.4)
+		(layer "F.Cu")
+		(net 15)
+	)
+	(segment
+		(start 143.15 95.7)
+		(end 143.2 95.65)
+		(width 0.4)
+		(layer "F.Cu")
+		(net 15)
+	)
+	(segment
+		(start 142.9 99.85)
+		(end 142.9 101.75)
+		(width 0.4)
+		(layer "F.Cu")
+		(net 15)
+	)
+	(segment
+		(start 145 99.55)
+		(end 143.2 99.55)
+		(width 0.4)
+		(layer "F.Cu")
+		(net 15)
+	)
+	(segment
+		(start 143.2 95.65)
+		(end 143.2 93.747316)
+		(width 0.4)
+		(layer "F.Cu")
+		(net 15)
+	)
+	(segment
+		(start 142.9 102.5)
+		(end 145.3 104.9)
 		(width 0.4)
 		(layer "F.Cu")
@@
 		(start 153.2 88.9)
 		(end 153.2 90.55)
-		(width 0.4)
+		(width 0.5)
 		(layer "F.Cu")
 		(net 15)
@@
 		(start 154.6 103.4)
 		(end 153.1 104.9)
-		(width 0.4)
-		(layer "F.Cu")
-		(net 15)
-	)
-	(segment
-		(start 143.585211 97.385211)
-		(end 143.585211 98.085211)
+		(width 0.5)
+		(layer "F.Cu")
+		(net 15)
+	)
+	(segment
+		(start 143.2 97.7)
+		(end 143.2 95.75)
+		(width 0.4)
+		(layer "F.Cu")
+		(net 15)
+	)
+	(segment
+		(start 143.2 93.747316)
+		(end 145.947316 91)
+		(width 0.4)
+		(layer "F.Cu")
+		(net 15)
+	)
+	(segment
+		(start 143.2 97.7)
+		(end 143.245 97.655)
+		(width 0.4)
+		(layer "F.Cu")
+		(net 15)
+	)
+	(segment
+		(start 143.245 97.655)
+		(end 145.025 97.655)
 		(width 0.4)
 		(layer "F.Cu")
@@
 		(start 158.6 104.2)
 		(end 158.3 104.5)
-		(width 0.4)
+		(width 0.5)
 		(layer "B.Cu")
 		(net 15)
@@
 		(start 158.3 103.4)
 		(end 158.6 103.7)
-		(width 0.4)
+		(width 0.5)
 		(layer "B.Cu")
 		(net 15)
@@
 	)
 	(segment
-		(start 157.5 86.25)
-		(end 155.85 84.6)
-		(width 0.4)
+		(start 151.75 92)
+		(end 151.2 92.55)
+		(width 0.4)
+		(layer "B.Cu")
+		(net 15)
+	)
+	(segment
+		(start 156.25 85)
+		(end 157.5 86.25)
+		(width 0.5)
 		(layer "B.Cu")
 		(net 15)
@@
 	)
 	(segment
-		(start 151.75 92)
-		(end 150.4 92)
+		(start 151.2 93.1)
+		(end 151.2 93.3)
 		(width 0.4)
 		(layer "B.Cu")
@@
 	)
 	(segment
-		(start 150.4 92)
-		(end 150.35 92.05)
-		(width 0.4)
-		(layer "B.Cu")
-		(net 15)
-	)
-	(segment
 		(start 156.25 103.4)
 		(end 158.3 103.4)
-		(width 0.4)
+		(width 0.5)
 		(layer "B.Cu")
 		(net 15)
@@
 	)
 	(segment
-		(start 150.35 92.05)
-		(end 150.35 93)
-		(width 0.4)
-		(layer "B.Cu")
-		(net 15)
-	)
-	(segment
-		(start 150.9 93)
-		(end 150.35 93)
+		(start 151.2 93.1)
+		(end 151.1 93)
 		(width 0.4)
 		(layer "B.Cu")
@@
 		(start 158.6 103.7)
 		(end 158.6 104.2)
-		(width 0.4)
+		(width 0.5)
 		(layer "B.Cu")
 		(net 15)
@@
 	)
 	(segment
+		(start 151.1 93)
+		(end 150.35 93)
+		(width 0.4)
+		(layer "B.Cu")
+		(net 15)
+	)
+	(segment
 		(start 151.2 101.6125)
 		(end 151.2 97)
@@
 	)
 	(segment
+		(start 155.25 85)
+		(end 156.25 85)
+		(width 0.5)
+		(layer "B.Cu")
+		(net 15)
+	)
+	(segment
+		(start 151.2 92.55)
+		(end 151.2 93.1)
+		(width 0.4)
+		(layer "B.Cu")
+		(net 15)
+	)
+	(segment
 		(start 152 102.4125)
 		(end 151.2 101.6125)
@@
 	)
 	(segment
-		(start 151.2 93.3)
-		(end 150.9 93)
-		(width 0.4)
-		(layer "B.Cu")
-		(net 15)
-	)
-	(segment
-		(start 155.85 84.6)
-		(end 155.25 84.6)
-		(width 0.4)
-		(layer "B.Cu")
-		(net 15)
-	)
-	(segment
 		(start 158.3 104.5)
 		(end 156.7 104.5)
-		(width 0.4)
-		(layer "B.Cu")
-		(net 15)
+		(width 0.5)
+		(layer "B.Cu")
+		(net 15)
