File: LumiTimeV2/PCB/KiCad/LumiTimeV2.kicad_pcb (KiCad board)
At the start: 2 copper layers, 35 x 35 mm, 54 parts, among them J1 Conn_06_Pin, U1 ATmega328-A, U2 PCF8563T, Y1 32,768 kHz

Commit message: Change#008
Add OSHW logo
Parts:
- removed D15: LL4148, Diode_SMD:D_MiniMELF
- added ZD1: BZV55C4V7, Diode_SMD:D_MiniMELF, B.Cu at (146.5, 84.9)
- D13: value BZV55C4V7 -> LL4148
- moved D14 7.37 mm to (146.5, 87.3), turned to 0 degrees
- moved D13 7.00 mm to (153.5, 85.1)
Connections:
- D13 pad 1: Net-(D13-K) -> +3V7
- D13 pad 2: GND -> Net-(D13-A)
- D14 pad 1: +3V7 -> /RXD
- D14 pad 2: Net-(D13-K) -> Net-(D13-A)
- PV12 pad 2: Net-(D13-K) -> Net-(D13-A)
Routing:
- net Net-(D13-K): track 9.35 -> 0.00 mm, vias 1 -> 0
- net Net-(D13-A): track 0.00 -> 9.35 mm, vias 0 -> 1
- net /But0: track 72.6 -> 72.1 mm
