File: LumiTimeV2/PCB/KiCad/LumiTimeV2.kicad_sch (KiCad schematic)
At the start: 54 parts, among them J1 Conn_06_Pin, U1 ATmega328-A, U2 PCF8563T, Y1 32,768 kHz

Commit message: Change#008
Add OSHW logo
Parts:
- BT1: value LIR2430 -> LIR3032
- renumbered D14 to D13, D15 to D14, D13 to ZD1
